Commit message: Added camera into the xarco, updated urdf_viewer and Sim_vs_Real_topics.md

File: robots/descriptions/go2_description/xacro/gazebo.xacro (robot description, xacro)
@@ -187,3 +187,37 @@
         <kd>1.0</kd>
     </gazebo>
+    <!-- Front RGB camera -->
+    <gazebo reference="camera_link">
+        <sensor name="camera_sensor" type="camera">
+            <always_on>true</always_on>
+            <visualize>true</visualize>
+            <update_rate>15.0</update_rate>
+            <camera>
+                <horizontal_fov>1.3962634</horizontal_fov>
+                <image>
+                    <width>640</width>
+                    <height>480</height>
+                    <format>R8G8B8</format>
+                </image>
+                <clip>
+                    <near>0.05</near>
+                    <far>30.0</far>
+                </clip>
+                <noise>
+                    <type>gaussian</type>
+                    <mean>0.0</mean>
+                    <stddev>0.0</stddev>
+                </noise>
+            </camera>
+            <plugin
+                name="camera_controller"
+                filename="libgazebo_ros_camera.so">
+                <ros>
+                    <namespace>/camera</namespace>
+                </ros>
+                <camera_name></camera_name>
+                <frame_name>camera_optical_frame</frame_name>
+            </plugin>
+        </sensor>
+    </gazebo>
 </robot>

File: robots/descriptions/go2_description/xacro/robot_VLP.xacro (robot description, xacro)
@@ -80,4 +80,41 @@
         </collision>
     </link>
+        <!-- Front RGB camera -->
+    <joint name="camera_joint" type="fixed">
+        <parent link="trunk"/>
+        <child link="camera_link"/>
+        <!-- Front of the robot, approximately at head/camera height -->
+        <origin xyz="0.32 0 0.04" rpy="0 0.0 0"/>
+    </joint>
+    <link name="camera_link">
+        <inertial>
+            <mass value="0.001"/>
+            <origin xyz="0 0 0" rpy="0 0 0"/>
+            <inertia
+                ixx="0.0001" ixy="0" ixz="0"
+                iyy="0.0001" iyz="0"
+                izz="0.0001"/>
+        </inertial>
+        <visual>
+            <origin xyz="0 0 0" rpy="0 0 0"/>
+            <geometry>
+                <box size="0.03 0.03 0.03"/>
+            </geometry>
+        </visual>
+        <collision>
+            <origin xyz="0 0 0" rpy="0 0 0"/>
+            <geometry>
+                <box size="0.03 0.03 0.03"/>
+            </geometry>
+        </collision>
+    </link>
+    <joint name="camera_optical_joint" type="fixed">
+        <parent link="camera_link"/>
+        <child link="camera_optical_frame"/>
+        <origin
+            xyz="0 0 0"
+            py="-1.57079632679 0 -1.57079632679"/>
+    </joint>
+    <link name="camera_optical_frame"/>
     <!--
     <joint name="load_joint" type="fixed">
